File: midi_cv_gate_v1_test_v1.kicad_pcb (KiCad board)
At the start: 2 copper layers, 90 x 100 mm, 170 parts, among them J1 Conn_01x20, J101 Conn_02x05_Odd_Even, J2 Conn_01x08, J3 Conn_01x20, U1 LM4040DBZ-5, U101 MCP3208, U102 MCP3208, U103 ARDUINO_PRO_MINI_custom_2, U104 MCP23018_SP, U105 LM7805_TO220

Commit message: A little cleanup
Other:
- board text added: "+5VA"
- board text added: "LM4040"
Changed lines of the file:
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@@
     (property "Sheetname" "")
     (attr exclude_from_pos_files)
-    (fp_text reference "H2" (at 0 -3.85) (layer "F.SilkS")
+    (fp_text reference "H2" (at 0 -3.85) (layer "F.SilkS") hide
       (effects (font (size 1 1) (thickness 0.15)))
     )
@@
     (property "Sheetname" "")
     (attr exclude_from_pos_files)
-    (fp_text reference "H3" (at -2.22 3.65) (layer "F.SilkS")
+    (fp_text reference "H3" (at -2.22 3.65) (layer "F.SilkS") hide
       (effects (font (size 1 1) (thickness 0.15)))
     )
@@
     (property "Sheetname" "")
     (attr exclude_from_pos_files)
-    (fp_text reference "H4" (at 0 -3.85) (layer "F.SilkS")
+    (fp_text reference "H4" (at 0 -3.85) (layer "F.SilkS") hide
       (effects (font (size 1 1) (thickness 0.15)))
     )
@@
     (property "Sheetname" "analog_inputs")
     (attr exclude_from_pos_files)
-    (fp_text reference "TP1" (at -3.17 0.07) (layer "F.SilkS")
+    (fp_text reference "TP1" (at -3.17 0.07) (layer "F.SilkS") hide
       (effects (font (size 1 1) (thickness 0.15)))
     )
@@
     (property "Sheetname" "")
     (attr exclude_from_pos_files)
-    (fp_text reference "H1" (at 3.34 3.02) (layer "F.SilkS")
+    (fp_text reference "H1" (at 3.34 3.02) (layer "F.SilkS") hide
       (effects (font (size 1 1) (thickness 0.15)))
     )
@@
     (effects (font (size 1 1) (thickness 0.15)) (justify mirror))
   )
-  (gr_text "ANALOG 5" (at 221 92.712006) (layer "B.SilkS")
+  (gr_text "ANALOG 5" (at 221.47619 92.712006) (layer "B.SilkS")
     (effects (font (size 1 1) (thickness 0.15)) (justify mirror))
   )
-  (gr_text "DIGITAL 7" (at 148.72 97.85) (layer "B.SilkS")
+  (gr_text "DIGITAL 7" (at 149.196191 97.85) (layer "B.SilkS")
     (effects (font (size 1 1) (thickness 0.15)) (justify mirror))
   )
@@
     (effects (font (size 1 1) (thickness 0.15)) (justify mirror))
   )
-  (gr_text "ANALOG 6" (at 221 95.260672) (layer "B.SilkS")
+  (gr_text "ANALOG 6" (at 221.47619 95.260672) (layer "B.SilkS")
     (effects (font (size 1 1) (thickness 0.15)) (justify mirror))
   )
-  (gr_text "ANALOG 8" (at 221 100.358004) (layer "B.SilkS")
+  (gr_text "ANALOG 8" (at 221.47619 100.358004) (layer "B.SilkS")
     (effects (font (size 1 1) (thickness 0.15)) (justify mirror))
   )
@@
     (effects (font (size 1 1) (thickness 0.15)) (justify mirror))
   )
-  (gr_text "DIGITAL 6" (at 148.72 95.31) (layer "B.SilkS")
+  (gr_text "DIGITAL 6" (at 149.196191 95.31) (layer "B.SilkS")
     (effects (font (size 1 1) (thickness 0.15)) (justify mirror))
   )
@@
     (effects (font (size 1 1) (thickness 0.15)) (justify mirror))
   )
-  (gr_text "DIGITAL 3" (at 148.72 87.69) (layer "B.SilkS")
+  (gr_text "DIGITAL 3" (at 149.196191 87.69) (layer "B.SilkS")
     (effects (font (size 1 1) (thickness 0.15)) (justify mirror))
   )
@@
     (effects (font (size 1 1) (thickness 0.15)) (justify mirror))
   )
+  (gr_text "+5VA" (at 180.94 86.43) (layer "B.SilkS")
+    (effects (font (size 1 1) (thickness 0.15)) (justify mirror))
+  )
   (gr_text "MCP3208" (at 196.81 101.68 90) (layer "B.SilkS")
     (effects (font (size 1 1) (thickness 0.15)) (justify mirror))
@@
     (effects (font (size 1 1) (thickness 0.15)) (justify mirror))
   )
-  (gr_text "DIGITAL 8" (at 148.72 100.39) (layer "B.SilkS")
+  (gr_text "DIGITAL 8" (at 149.196191 100.39) (layer "B.SilkS")
     (effects (font (size 1 1) (thickness 0.15)) (justify mirror))
   )
@@
     (effects (font (size 1 1) (thickness 0.15)) (justify mirror))
   )
-  (gr_text "ANALOG 7" (at 221 97.809338) (layer "B.SilkS")
+  (gr_text "ANALOG 7" (at 221.47619 97.809338) (layer "B.SilkS")
     (effects (font (size 1 1) (thickness 0.15)) (justify mirror))
   )
@@
     (effects (font (size 1 1) (thickness 0.15)) (justify mirror))
   )
-  (gr_text "ANALOG 2" (at 221 85.066008) (layer "B.SilkS")
+  (gr_text "ANALOG 2" (at 221.47619 85.066008) (layer "B.SilkS")
     (effects (font (size 1 1) (thickness 0.15)) (justify mirror))
   )
@@
     (effects (font (size 1 1) (thickness 0.15)) (justify mirror))
   )
-  (gr_text "ANALOG 9" (at 221 102.90667) (layer "B.SilkS")
+  (gr_text "ANALOG 9" (at 221.47619 102.90667) (layer "B.SilkS")
     (effects (font (size 1 1) (thickness 0.15)) (justify mirror))
   )
-  (gr_text "DIGITAL 4" (at 148.72 90.23) (layer "B.SilkS")
+  (gr_text "DIGITAL 4" (at 149.196191 90.23) (layer "B.SilkS")
     (effects (font (size 1 1) (thickness 0.15)) (justify mirror))
   )
-  (gr_text "DIGITAL 5" (at 148.72 92.77) (layer "B.SilkS")
+  (gr_text "DIGITAL 5" (at 149.196191 92.77) (layer "B.SilkS")
     (effects (font (size 1 1) (thickness 0.15)) (justify mirror))
   )
@@
     (effects (font (size 1 1) (thickness 0.15)) (justify mirror))
   )
-  (gr_text "ANALOG 3" (at 221 87.614674) (layer "B.SilkS")
+  (gr_text "ANALOG 3" (at 221.47619 87.614674) (layer "B.SilkS")
     (effects (font (size 1 1) (thickness 0.15)) (justify mirror))
   )
-  (gr_text "DIGITAL 2" (at 148.72 85.15) (layer "B.SilkS")
+  (gr_text "DIGITAL 2" (at 149.196191 85.15) (layer "B.SilkS")
     (effects (font (size 1 1) (thickness 0.15)) (justify mirror))
   )
@@
     (effects (font (size 1 1) (thickness 0.15)) (justify mirror))
   )
-  (gr_text "ANALOG 1" (at 221 82.517342) (layer "B.SilkS")
+  (gr_text "ANALOG 1" (at 221.47619 82.517342) (layer "B.SilkS")
     (effects (font (size 1 1) (thickness 0.15)) (justify mirror))
   )
@@
     (effects (font (size 1 1) (thickness 0.15)) (justify mirror))
   )
-  (gr_text "DIGITAL 1" (at 148.72 82.61) (layer "B.SilkS")
+  (gr_text "DIGITAL 1" (at 149.196191 82.61) (layer "B.SilkS")
     (effects (font (size 1 1) (thickness 0.15)) (justify mirror))
   )
-  (gr_text "ANALOG 4" (at 221 90.16334) (layer "B.SilkS")
+  (gr_text "ANALOG 4" (at 221.47619 90.16334) (layer "B.SilkS")
     (effects (font (size 1 1) (thickness 0.15)) (justify mirror))
   )
@@
     (effects (font (size 1 1) (thickness 0.15)) (justify mirror))
   )
-  (gr_text "DIGITAL 0" (at 148.72 80.07) (layer "B.SilkS")
+  (gr_text "DIGITAL 0" (at 149.196191 80.07) (layer "B.SilkS")
     (effects (font (size 1 1) (thickness 0.15)) (justify mirror))
   )
@@
     (effects (font (size 1 1) (thickness 0.15)) (justify mirror))
   )
-  (gr_text "DIGITAL 9" (at 148.72 102.93) (layer "B.SilkS")
+  (gr_text "DIGITAL 9" (at 149.196191 102.93) (layer "B.SilkS")
     (effects (font (size 1 1) (thickness 0.15)) (justify mirror))
   )
-  (gr_text "ANALOG 0" (at 221 79.968676) (layer "B.SilkS")
+  (gr_text "ANALOG 0" (at 221.47619 79.968676) (layer "B.SilkS")
     (effects (font (size 1 1) (thickness 0.15)) (justify mirror))
   )
@@
     (effects (font (size 1 1) (thickness 0.15)))
   )
+  (gr_text "LM4040" (at 181.05 90.85 90) (layer "F.SilkS")
+    (effects (font (size 1 1) (thickness 0.15)))
+  )
   (gr_text "RobotDialogs\n" (at 185 65.2) (layer "F.SilkS")
     (effects (font (size 1 1) (thickness 0.15)))
@@
     (effects (font (size 1 1) (thickness 0.15)))
   )
+  (gr_text "+5VA" (at 180.78 86.43) (layer "F.SilkS")
+    (effects (font (size 1 1) (thickness 0.15)))
+  )
