File: midi_cv_gate_v1_test_v1.kicad_pcb (KiCad board)
At the start: 2 copper layers, 90 x 100 mm, 170 parts, among them J1 Conn_01x20, J101 Conn_02x05_Odd_Even, J2 Conn_01x08, J3 Conn_01x20, U1 LM4040DBZ-5, U101 MCP3208, U102 MCP3208, U103 ARDUINO_PRO_MINI_custom_2, U104 MCP23018_SP, U105 LM7805_TO220

Commit message: Resync pcb and schematic
Parts:
- D101: value +5_LED -> LED3
- D102: value +5_LED -> LED2
- D103: value +5_LED -> LED1
