File: midi_cv_gate_v1_test_v1_analog_inputs.kicad_sch (KiCad schematic)
At the start: 81 parts, among them U3 MCP3208, U4 MCP3208, U6 LM4040DBZ-5

Commit message: First pass routing done
Parts:
- added JP8: Jumper_2_Open, Jumper:SolderJumper-2_P1.3mm_Open_Pad1.0x1.5mm, symbol Jumper:Jumper_2_Open
Connections:
- net +5V: now also JP8.2 (B)
- net +5VA: now also JP8.1 (A)
Other:
- moved on the sheet: TP1
Changed lines of the file:
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@@
   (junction (at 243.84 101.6) (diameter 0) (color 0 0 0 0)
   )
+  (junction (at 254 55.88) (diameter 0) (color 0 0 0 0)
+  )
   (junction (at 223.52 137.16) (diameter 0) (color 0 0 0 0)
   )
@@
     (stroke (width 0) (type default) (color 0 0 0 0))
   )
+  (wire (pts (xy 254 50.8) (xy 254 55.88))
+    (stroke (width 0) (type default) (color 0 0 0 0))
+  )
   (wire (pts (xy 45.72 53.34) (xy 40.64 53.34))
     (stroke (width 0) (type default) (color 0 0 0 0))
@@
   )
   (wire (pts (xy 152.4 58.42) (xy 170.18 58.42))
+    (stroke (width 0) (type default) (color 0 0 0 0))
+  )
+  (wire (pts (xy 254 60.96) (xy 254 55.88))
     (stroke (width 0) (type default) (color 0 0 0 0))
   )
@@
     (pin "1")
   )
-  (symbol (lib_id "Connector:TestPoint") (at 254 43.18 0) (unit 1)
-    (in_bom yes) (on_board yes) (fields_autoplaced)
-    (property "Reference" "TP1" (id 0) (at 255.397 38.9695 0)
-      (effects (font (size 1.27 1.27)) (justify left))
-    )
-    (property "Value" "TestPoint" (id 1) (at 255.397 41.7446 0)
-      (effects (font (size 1.27 1.27)) (justify left))
-    )
-    (property "Footprint" "TestPoint:TestPoint_THTPad_2.0x2.0mm_Drill1.0mm" (id 2) (at 259.08 43.18 0)
-      (effects (font (size 1.27 1.27)) hide)
-    )
-    (property "Datasheet" "~" (id 3) (at 259.08 43.18 0)
+  (symbol (lib_id "Connector:TestPoint") (at 254 50.8 0) (unit 1)
+    (in_bom yes) (on_board yes) (fields_autoplaced)
+    (property "Reference" "TP1" (id 0) (at 255.397 46.5895 0)
+      (effects (font (size 1.27 1.27)) (justify left))
+    )
+    (property "Value" "TestPoint" (id 1) (at 255.397 49.3646 0)
+      (effects (font (size 1.27 1.27)) (justify left))
+    )
+    (property "Footprint" "TestPoint:TestPoint_THTPad_2.0x2.0mm_Drill1.0mm" (id 2) (at 259.08 50.8 0)
+      (effects (font (size 1.27 1.27)) hide)
+    )
+    (property "Datasheet" "~" (id 3) (at 259.08 50.8 0)
       (effects (font (size 1.27 1.27)) hide)
     )
@@
     )
     (property "Datasheet" "~" (id 3) (at 194.31 50.8 0)
+      (effects (font (size 1.27 1.27)) hide)
+    )
+    (pin "1")
+    (pin "2")
+  )
+  (symbol (lib_id "Jumper:Jumper_2_Open") (at 259.08 55.88 0) (unit 1)
+    (in_bom yes) (on_board yes) (fields_autoplaced)
+    (property "Reference" "JP8" (id 0) (at 259.08 50.2625 0))
+    (property "Value" "Jumper_2_Open" (id 1) (at 259.08 53.0376 0))
+    (property "Footprint" "Jumper:SolderJumper-2_P1.3mm_Open_Pad1.0x1.5mm" (id 2) (at 259.08 55.88 0)
+      (effects (font (size 1.27 1.27)) hide)
+    )
+    (property "Datasheet" "~" (id 3) (at 259.08 55.88 0)
       (effects (font (size 1.27 1.27)) hide)
     )
@@
     (pin "2")
   )
+  (symbol (lib_id "power:+5V") (at 264.16 55.88 270) (unit 1)
+    (in_bom yes) (on_board yes) (fields_autoplaced)
+    (property "Reference" "#PWR021" (id 0) (at 260.35 55.88 0)
+      (effects (font (size 1.27 1.27)) hide)
+    )
+    (property "Value" "+5V" (id 1) (at 267.335 56.359 90)
+      (effects (font (size 1.27 1.27)) (justify left))
+    )
+    (property "Footprint" "" (id 2) (at 264.16 55.88 0)
+      (effects (font (size 1.27 1.27)) hide)
+    )
+    (property "Datasheet" "" (id 3) (at 264.16 55.88 0)
+      (effects (font (size 1.27 1.27)) hide)
+    )
+    (pin "1")
+  )
   (symbol (lib_id "power:+5V") (at 246.38 129.54 0) (unit 1)
     (in_bom yes) (on_board yes)
@@
     (pin "2")
   )
-  (symbol (lib_id "power:+5VA") (at 254 43.18 180) (unit 1)
-    (in_bom yes) (on_board yes) (fields_autoplaced)
-    (property "Reference" "#PWR040" (id 0) (at 254 39.37 0)
-      (effects (font (size 1.27 1.27)) hide)
-    )
-    (property "Value" "+5VA" (id 1) (at 255.397 44.929 0)
-      (effects (font (size 1.27 1.27)) (justify right))
-    )
-    (property "Footprint" "" (id 2) (at 254 43.18 0)
-      (effects (font (size 1.27 1.27)) hide)
-    )
-    (property "Datasheet" "" (id 3) (at 254 43.18 0)
-      (effects (font (size 1.27 1.27)) hide)
-    )
+  (symbol (lib_id "power:+5VA") (at 254 60.96 180) (unit 1)
+    (in_bom yes) (on_board yes) (fields_autoplaced)
+    (property "Reference" "#PWR040" (id 0) (at 254 57.15 0)
+      (effects (font (size 1.27 1.27)) hide)
+    )
+    (property "Value" "+5VA" (id 1) (at 255.397 62.709 0)
+      (effects (font (size 1.27 1.27)) (justify right))
+    )
+    (property "Footprint" "" (id 2) (at 254 60.96 0)
+      (effects (font (size 1.27 1.27)) hide)
+    )
+    (property "Datasheet" "" (id 3) (at 254 60.96 0)
+      (effects (font (size 1.27 1.27)) hide)
+    )

Commit message: Geographic re-annotate
Parts:
- renumbered C16 to C10, C15 to C11, C14 to C12, C12 to C14, C20 to C15, C21 to C16, C22 to C17, C23 to C18, C24 to C19, C25 to C20, C26 to C21, C27 to C22, C10 to C5, C8 to C6, C19 to C7, C18 to C8, C17 to C9, JP8 to JP5, R30 to R100, R28 to R101, R26 to R102, R24 to R103, R22 to R104, R20 to R105, R18 to R106, R16 to R107, R102 to R108, R104 to R109, R106 to R110, R108 to R111, R110 to R112, R112 to R113, R116 to R115, R117 to R53, R47 to R56, R51 to R57, R48 to R58, R49 to R59, R50 to R60, R52 to R61, R56 to R62, R53 to R63, R54 to R64, R55 to R65, R38 to R68, R29 to R69, R37 to R70, R27 to R71, R36 to R72, R25 to R73, R35 to R74, R23 to R75, R34 to R76, R21 to R77, R33 to R78, R19 to R79, R32 to R80, R17 to R81, R31 to R82, R15 to R83, R39 to R84, R101 to R85, R40 to R86, R103 to R87, R41 to R88, R105 to R89, R42 to R90, R107 to R91, R43 to R92, R109 to R93, R44 to R94, R111 to R95, R45 to R96, R113 to R97, R46 to R98, R115 to R99, U6 to U1, U3 to U101, U4 to U102

Commit message: Resync pcb and schematic
Other:
- note added: "Pull MISO (Dout) Low, it's HIGH-Z and we want 0's. Pull CS HIGH."
- company: (none) -> RobotDialogs
- title: (none) -> MIDI CV GATE Test Fixture
Changed lines of the file:
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@@
 (kicad_sch (version 20211123) (generator eeschema)
   (paper "A4")
+  (title_block
+    (title "MIDI CV GATE Test Fixture")
+    (date "2022-10-15")
+    (rev "1.0")
+    (company "RobotDialogs")
+  )
   (junction (at 121.92 124.46) (diameter 0) (color 0 0 0 0)
   )
@@
     (effects (font (size 1.27 1.27)) (justify left bottom))
   )
+  (text "Pull MISO (Dout) Low, it's HIGH-Z and we want 0's.\nPull CS HIGH."
+    (at 220.98 155.575 0)
+    (effects (font (size 1.27 1.27)) (justify left bottom))
+  )

Commit message: Component updates and rework info v1
Parts:
- R57, R58, R59, R61, R62, R64, R65: value 10k -> DNU
Changed lines of the file:
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@@
       (effects (font (size 1.27 1.27)) (justify left))
     )
-    (property "Value" "10k" (id 1) (at 225.298 142.8366 0)
+    (property "Value" "DNU" (id 1) (at 225.298 142.8366 0)
       (effects (font (size 1.27 1.27)) (justify left))
     )
@@
       (effects (font (size 1.27 1.27)) (justify left))
     )
-    (property "Value" "10k" (id 1) (at 232.41 135.7441 0)
+    (property "Value" "DNU" (id 1) (at 232.41 135.7441 0)
       (effects (font (size 1.27 1.27)) (justify left))
     )
@@
       (effects (font (size 1.27 1.27)) (justify left))
     )
-    (property "Value" "10k" (id 1) (at 240.03 135.4901 0)
+    (property "Value" "DNU" (id 1) (at 240.03 135.4901 0)
       (effects (font (size 1.27 1.27)) (justify left))
     )
@@
       (effects (font (size 1.27 1.27)) (justify left))
     )
-    (property "Value" "10k" (id 1) (at 232.918 143.0906 0)
+    (property "Value" "DNU" (id 1) (at 232.918 143.0906 0)
       (effects (font (size 1.27 1.27)) (justify left))
     )
@@
       (effects (font (size 1.27 1.27)) (justify left))
     )
-    (property "Value" "10k" (id 1) (at 247.65 142.748 0)
+    (property "Value" "DNU" (id 1) (at 247.65 142.748 0)
       (effects (font (size 1.27 1.27)) (justify left))
     )
@@
       (effects (font (size 1.27 1.27)) (justify left))
     )
-    (property "Value" "10k" (id 1) (at 247.65 135.128 0)
+    (property "Value" "DNU" (id 1) (at 247.65 135.128 0)
       (effects (font (size 1.27 1.27)) (justify left))
     )
@@
       (effects (font (size 1.27 1.27)) (justify left))
     )
-    (property "Value" "10k" (id 1) (at 255.778 142.8366 0)
-      (effects (font (size 1.27 1.27)) (justify left))
-    )
+    (property "Value" "DNU" (id 1) (at 255.778 142.8366 0)
+      (effects (font (size 1.27 1.27)) (justify left))
+    )
