File: midi_cv_gate_v1_test_v1_digital_io.kicad_sch (KiCad schematic)
At the start: 46 parts, among them U5 MCP23018_SP

Commit message: Geographic re-annotate
Parts:
- renumbered C11 to C4, R100 to R1, R59 to R10, R61 to R11, R63 to R12, R65 to R13, R67 to R14, R69 to R15, R71 to R16, R98 to R2, R99 to R20, R97 to R21, R95 to R22, R93 to R23, R91 to R24, R89 to R25, R87 to R26, R85 to R27, R58 to R28, R60 to R29, R96 to R3, R62 to R30, R64 to R31, R66 to R32, R68 to R33, R70 to R34, R72 to R35, R84 to R39, R94 to R4, R78 to R40, R83 to R42, R77 to R43, R76 to R44, R82 to R45, R75 to R46, R81 to R47, R92 to R5, R74 to R50, R73 to R51, R80 to R54, R79 to R55, R90 to R6, R88 to R7, R86 to R8, R57 to R9, U5 to U104

Commit message: Resync pcb and schematic
Other:
- company: (none) -> RobotDialogs
- title: (none) -> MIDI CV GATE Test Fixture
Changed lines of the file:
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@@
 (kicad_sch (version 20211123) (generator eeschema)
   (paper "A4")
+  (title_block
+    (title "MIDI CV GATE Test Fixture")
+    (date "2022-10-15")
+    (rev "1.0")
+    (company "RobotDialogs")
+  )
   (junction (at 205.74 121.92) (diameter 0) (color 0 0 0 0)
   )

Commit message: Component updates and rework info v1
Parts:
- R40, R42, R44, R46, R54, R55: value 10k -> DNU
Changed lines of the file:
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@@
       (effects (font (size 1.27 1.27)) (justify left))
     )
-    (property "Value" "10k" (id 1) (at 133.858 117.4366 0)
+    (property "Value" "DNU" (id 1) (at 133.858 117.4366 0)
       (effects (font (size 1.27 1.27)) (justify left))
     )
@@
       (effects (font (size 1.27 1.27)) (justify left))
     )
-    (property "Value" "10k" (id 1) (at 118.11 117.475 0)
+    (property "Value" "DNU" (id 1) (at 118.11 117.475 0)
       (effects (font (size 1.27 1.27)) (justify left))
     )
@@
       (effects (font (size 1.27 1.27)) (justify left))
     )
-    (property "Value" "10k" (id 1) (at 95.758 125.0566 0)
+    (property "Value" "DNU" (id 1) (at 95.758 125.0566 0)
       (effects (font (size 1.27 1.27)) (justify left))
     )
@@
       (effects (font (size 1.27 1.27)) (justify left))
     )
-    (property "Value" "10k" (id 1) (at 110.49 117.475 0)
+    (property "Value" "DNU" (id 1) (at 110.49 117.475 0)
       (effects (font (size 1.27 1.27)) (justify left))
     )
@@
       (effects (font (size 1.27 1.27)) (justify left))
     )
-    (property "Value" "10k" (id 1) (at 103.378 125.0566 0)
+    (property "Value" "DNU" (id 1) (at 103.378 125.0566 0)
       (effects (font (size 1.27 1.27)) (justify left))
     )
@@
       (effects (font (size 1.27 1.27)) (justify left))
     )
-    (property "Value" "10k" (id 1) (at 126.238 125.0566 0)
-      (effects (font (size 1.27 1.27)) (justify left))
-    )
+    (property "Value" "DNU" (id 1) (at 126.238 125.0566 0)
+      (effects (font (size 1.27 1.27)) (justify left))
+    )
